File: MCU_Datalogger.kicad_pcb (KiCad board)
At the start: 2 copper layers, 29 parts, among them J1 Conn_01x04_Male, J2 Conn_01x09_Male, J3 Conn_01x04_Male, J4 Conn_02x03_Odd_Even, U1 24LC1025, U2 DS1337S+, U3 24LC1025, U4 ATMEGA328P-AU, Y1 32.768KHz, Y2 16MHz

Commit message: commit3
Parts:
- moved H3 77.0 mm to (206.0, 61.0), turned to 90 degrees
- moved U4 74.3 mm to (177.5, 71.4)
- moved H2 60.4 mm to (206.0, 89.5), turned to 90 degrees
- moved D1 58.2 mm to (195.6, 62.3)
- moved C4 48.8 mm to (185.2, 75.7)
- moved R3 48.7 mm to (192.1, 67.6)
- moved C5 48.5 mm to (182.1, 63.6)
- moved R7 44.9 mm to (192.0, 64.4), turned to 180 degrees
- moved R6 44.2 mm to (192.1, 70.8)
- moved C2 44.1 mm to (185.0, 79.2)
- moved C1 43.0 mm to (173.1, 63.3)
- moved Y2 40.5 mm to (177.9, 79.2)
- moved R4 40.3 mm to (195.5, 67.6)
- moved U3 39.0 mm to (163.6, 70.7)
- moved D2 37.8 mm to (192.1, 62.3)
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Connections:
- BT1 pad 1: Net-(BT1-Pad1) -> /Vcc
- C5 pad 1: Net-(BT1-Pad1) -> /Vcc
- D2 pad 2: Net-(BT1-Pad1) -> /Vcc
- J1 pad 1: unconnected-(J1-Pad1) -> GND
- J1 pad 2: unconnected-(J1-Pad2) -> /Vcc
- J1 pad 3: unconnected-(J1-Pad3) -> /SDA
- J1 pad 4: unconnected-(J1-Pad4) -> /SCK
- J2 pad 1: unconnected-(J2-Pad1) -> /D2
- J2 pad 2: unconnected-(J2-Pad2) -> /D3
- J2 pad 3: unconnected-(J2-Pad3) -> /D4
- J2 pad 4: unconnected-(J2-Pad4) -> /D5
- J2 pad 5: unconnected-(J2-Pad5) -> /D6
- J2 pad 6: unconnected-(J2-Pad6) -> /D7
- J2 pad 7: unconnected-(J2-Pad7) -> /D8
- J2 pad 8: unconnected-(J2-Pad8) -> GND
- J2 pad 9: unconnected-(J2-Pad9) -> /Vcc
- J3 pad 1: unconnected-(J3-Pad1) -> GND
- J3 pad 2: unconnected-(J3-Pad2) -> /Vcc
- J3 pad 3: unconnected-(J3-Pad3) -> /RX
- J3 pad 4: unconnected-(J3-Pad4) -> /TX
- J4 pad 1: unconnected-(J4-Pad1) -> /MISO
- J4 pad 2: unconnected-(J4-Pad2) -> /Vcc
- J4 pad 3: unconnected-(J4-Pad3) -> /SCK
- J4 pad 4: unconnected-(J4-Pad4) -> /MOSI
- J4 pad 5: unconnected-(J4-Pad5) -> /RESET
- J4 pad 6: unconnected-(J4-Pad6) -> GND
- U4 pad 18: Net-(BT1-Pad1) -> /Vcc
- U4 pad 4: unconnected-(U4-Pad4) -> /Vcc
Routing:
- net /Vcc: track 0.00 -> 157.9 mm, vias 0 -> 7
- net GND: track 0.00 -> 143.7 mm, vias 0 -> 12
- net /SDA: track 0.00 -> 60.2 mm, vias 0 -> 4
- net /SCK: track 0.00 -> 41.2 mm, vias 0 -> 2
- net /D3: track 0.00 -> 38.0 mm, vias 0 -> 2
- net /D2: track 0.00 -> 37.1 mm, vias 0 -> 2
- net /D4: track 0.00 -> 29.6 mm, vias 0 -> 2
- net /D5: track 0.00 -> 21.2 mm, vias 0 -> 2
- net /D6: track 0.00 -> 19.7 mm, vias 0 -> 2
- net Net-(C2-Pad2): track 0.00 -> 18.6 mm, vias 0 -> 2
- net /D7: track 0.00 -> 18.6 mm, vias 0 -> 2
- net /D8: track 0.00 -> 17.2 mm, vias 0 -> 2
- net /RX: track 0.00 -> 13.5 mm, vias 0 -> 2
- net Net-(C4-Pad2): track 0.00 -> 11.2 mm
- net Net-(R2-Pad2): track 0.00 -> 10.1 mm
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Other:
- board outline added: 62.4 x 36.3 mm

Commit message: tekrar
Parts:
- added REF**: logo_1, ayprologo:logo_1, F.Cu at (198.9, 87.7)
- turned R4 to 180 degrees
- turned R5 to 180 degrees
Routing:
- net /SCK: track 41.2 -> 117.0 mm, vias 2 -> 9
- net /MISO: track 0.00 -> 59.3 mm, vias 0 -> 3
- net /MOSI: track 0.00 -> 47.9 mm, vias 0 -> 3
- net /TX: track 0.00 -> 33.3 mm, vias 0 -> 3
- net /SDA: track 60.2 -> 85.5 mm, vias 4 -> 8
- net /RESET: track 2.53 -> 27.5 mm, vias 1 -> 3
- net /RX: track 13.5 -> 33.4 mm, vias 2 -> 3
- net /Vcc: track 157.9 -> 172.1 mm, vias 7 -> 9
- net GND: track 143.7 -> 157.8 mm
- net Net-(D1-Pad1): track 2.83 -> 2.13 mm
Other:
- board size 62.4 x 36.3 mm -> 62.4 x 36.4 mm

Commit message: commit 2
Parts:
- moved J1 84.8 mm to (264.2, 66.0), turned to 0 degrees
- moved BT1 81.1 mm to (235.9, 77.6)
- moved R1 80.5 mm to (244.9, 74.6), turned to 0 degrees
- moved R2 79.7 mm to (240.5, 74.7)
- moved C3 77.8 mm to (247.0, 65.2), turned to 0 degrees
- moved J4 74.3 mm to (273.5, 66.0)
- moved J3 69.1 mm to (268.9, 66.0), turned to 0 degrees
- moved C1 60.0 mm to (230.0, 82.1)
- moved R6 59.6 mm to (251.4, 65.1)
- moved R3 54.9 mm to (247.0, 68.2)
- moved C2 53.1 mm to (237.6, 71.7)
- moved R7 50.6 mm to (242.1, 71.7), turned to 0 degrees
- moved C5 47.2 mm to (224.1, 85.1)
- moved R5 43.6 mm to (234.5, 84.0), turned to 0 degrees
- moved J2 41.9 mm to (190.0, 63.0), turned to -90 degrees
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Routing:
- net /Vcc: track 172.1 -> 0.00 mm, vias 9 -> 0
- net GND: track 157.8 -> 0.00 mm, vias 12 -> 0
- net /SCK: track 117.0 -> 0.00 mm, vias 9 -> 0
- net /SDA: track 85.5 -> 0.00 mm, vias 8 -> 0
- net /MISO: track 59.3 -> 0.00 mm, vias 3 -> 0
- net /MOSI: track 47.9 -> 0.00 mm, vias 3 -> 0
- net /D3: track 38.0 -> 0.00 mm, vias 2 -> 0
- net /D2: track 37.1 -> 0.00 mm, vias 2 -> 0
- net /RX: track 33.4 -> 0.00 mm, vias 3 -> 0
- net /TX: track 33.3 -> 0.00 mm, vias 3 -> 0
- net /D4: track 29.6 -> 0.00 mm, vias 2 -> 0
- net /RESET: track 27.5 -> 0.00 mm, vias 3 -> 0
- net /D5: track 21.2 -> 0.00 mm, vias 2 -> 0
- net /D6: track 19.7 -> 0.00 mm, vias 2 -> 0
- net Net-(C2-Pad2): track 18.6 -> 0.00 mm, vias 2 -> 0
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